Commit message: Updates Ridgeback integration

File: src/baxter/baxter_common/baxter_description/urdf/baxter.urdf.xacro (robot description, xacro)
@@ -3,6 +3,6 @@
   <xacro:arg name="gazebo" default="false"/>
   <!-- Arg for choosing default pedestal or Baxter-Ridgeback mounting -->
-  <xacro:arg name="pedestal" default="true"/>
-  <xacro:arg name="pedestal_ridgeback" default="false"/>
+  <xacro:arg name="pedestal" default="false"/>
+  <xacro:arg name="pedestal_ridgeback" default="true"/>
   <xacro:arg name="right_electric_gripper" default="true"/>
   <xacro:arg name="left_electric_gripper" default="true"/>

File: src/ridgeback_baxter/ridgeback_baxter_description/urdf/ridgeback_baxter.urdf (robot description, URDF)
Before this commit: robot ridgeback_baxter, 75 links, 74 joints
Links:
- added link front_laser, mass 0.130; collision box size=0.05 0.05 0.07; visual mesh filename=package://ridgeback_description/meshes/ust-10lx.stl
- added link rear_laser, mass 0.130; collision box size=0.05 0.05 0.07; visual mesh filename=package://ridgeback_description/meshes/ust-10lx.stl
- link l_gripper_l_finger: geometry collision box size=0.01 0.0135 0.075; collision box size=0.01 0.05 0.017
- link l_gripper_l_finger_tip: geometry collision box size=0.016 0.007 0.037; visual mesh filename=package://rethink_ee_description/meshes/electric_gripper/fi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
- link l_gripper_r_finger: geometry collision box size=0.01 0.0135 0.075; collision box size=0.01 0.05 0.017
- link l_gripper_r_finger_tip: geometry collision box size=0.016 0.007 0.037; visual mesh filename=package://rethink_ee_description/meshes/electric_gripper/fi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
- link r_gripper_l_finger: geometry collision box size=0.01 0.0135 0.1127; collision box size=0.01 0.08778 0.017
- link r_gripper_l_finger_tip: geometry collision box size=0.042 0.0065 0.037; visual mesh filename=package://rethink_ee_description/meshes/electric_gripper/fi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
- link r_gripper_r_finger: geometry collision box size=0.01 0.0135 0.1127; collision box size=0.01 0.08778 0.017
- link r_gripper_r_finger_tip: geometry collision box size=0.042 0.0065 0.037; visual mesh filename=package://rethink_ee_description/meshes/electric_gripper/fi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
Joints:
- added joint front_laser_joint: type fixed, parent chassis_link, child front_laser, origin xyz=0.3932 0 0.2330 rpy=0 0 0.0
- added joint rear_laser_joint: type fixed, parent chassis_link, child rear_laser, origin xyz=-0.3932 0 0.2330 rpy=0 0 3.14159265359
- joint l_gripper_l_finger_joint: origin xyz=0.0 -0.0015 0.02 rpy=0 0 0 -> xyz=0.0 -0.011 0.02 rpy=0 0 0
- joint l_gripper_l_finger_tip_joint: origin xyz=0.0 0.01725 0.1127 rpy=0 0 0 -> xyz=0.0 0.01725 0.075 rpy=0 0 0
- joint l_gripper_r_finger_joint: origin xyz=0.0 0.0015 0.02 rpy=0 0 0 -> xyz=0.0 0.011 0.02 rpy=0 0 0
- joint l_gripper_r_finger_tip_joint: origin xyz=0.0 -0.01725 0.1127 rpy=0 0 0 -> xyz=0.0 -0.01725 0.075 rpy=0 0 0
- joint left_endpoint: origin xyz=0 0 0.1327 rpy=0 0 0 -> xyz=0 0 0.095 rpy=0 0 0
- joint r_gripper_l_finger_joint: origin xyz=0.0 -0.011 0.02 rpy=0 0 0 -> xyz=0.0 0.0175 0.02 rpy=0 0 0
- joint r_gripper_l_finger_tip_joint: origin xyz=0.0 0.01725 0.075 rpy=0 0 0 -> xyz=0.0 0.05503 0.1127 rpy=0 0 0
- joint r_gripper_r_finger_joint: origin xyz=0.0 0.011 0.02 rpy=0 0 0 -> xyz=0.0 -0.0175 0.02 rpy=0 0 0
- joint r_gripper_r_finger_tip_joint: origin xyz=0.0 -0.01725 0.075 rpy=0 0 0 -> xyz=0.0 -0.05503 0.1127 rpy=0 0 0
- joint ridgeback_base_to_baxter: origin xyz=0.2 0 0.565 rpy=0 0 0 -> xyz=0.2 0 0.85 rpy=0 0 0; parent mid_mount -> chassis_link
- joint right_endpoint: origin xyz=0 0 0.095 rpy=0 0 0 -> xyz=0 0 0.1327 rpy=0 0 0

File: src/ridgeback_baxter/ridgeback_baxter_description/urdf/ridgeback_baxter.urdf.xacro (robot description, xacro)
@@ -5,11 +5,4 @@
   <!--Ridgeback Robot-->
   <xacro:include filename="$(find ridgeback_description)/urdf/ridgeback.urdf.xacro" />
-  <xacro:include filename="$(find ridgeback_description)/urdf/accessories/hokuyo_ust-10lx_mount.urdf.xacro" />
-    <xacro:hokuyo_ust-10lx_mount prefix="front"
-                                 topic="front/scan"
-                                 location="1" />
-    <xacro:hokuyo_ust-10lx_mount prefix="rear"
-                                 topic="rear/scan"
-                                 location="-1" />
   <!-- Baxter Robot -->
   <xacro:include filename="$(find baxter_description)/urdf/baxter.urdf.xacro" />
@@ -18,8 +11,8 @@
   <xacro:property name="pedestal_offset_x" value="0.2" />
   <!-- Link Baxter and Ridgeback-->
-  <joint name="ridgeback_base_to_baxter" type="fixed">
+  <!-- <joint name="ridgeback_base_to_baxter" type="fixed">
       <origin rpy="0 0 0" xyz="${pedestal_offset_x} 0 ${pedestal_height}" />
       <parent link="chassis_link" />
       <child link="base" />
-  </joint>
+  </joint> -->
 </robot>

Commit message: FINAL VERSION FOR INTEL NUC

File: src/baxter/baxter_common/baxter_description/urdf/baxter.urdf.xacro (robot description, xacro)
@@ -2,9 +2,5 @@
 <robot name="baxter" xmlns:xacro="http://www.ros.org/wiki/xacro">
   <xacro:arg name="gazebo" default="false"/>
-  <!-- Arg for choosing default pedestal or Baxter-Ridgeback mounting -->
-  <xacro:arg name="pedestal" default="false"/>
-  <xacro:arg name="pedestal_ridgeback" default="true"/>
-  <xacro:arg name="right_electric_gripper" default="true"/>
-  <xacro:arg name="left_electric_gripper" default="true"/>
+  <xacro:arg name="pedestal" default="true"/>
   <!-- Baxter Base URDF -->
   <xacro:include filename="$(find baxter_description)/urdf/baxter_base/baxter_base.urdf.xacro">
@@ -13,20 +9,11 @@
   <!-- Baxter Pedestal -->
   <xacro:if value="$(arg pedestal)">
-    <xacro:include filename="$(find baxter_description)/urdf/pedestal/pedestal_default.xacro">
-      <xacro:arg name="gazebo" value="${gazebo}"/>
-    </xacro:include>
-  </xacro:if>
-  <xacro:if value="$(arg pedestal_ridgeback)">
-    <xacro:include filename="$(find baxter_description)/urdf/pedestal/pedestal.xacro">
+    <xacro:include filename="$(find baxter_description)/urdf/pedestal/pedestal_u.xacro">
       <xacro:arg name="gazebo" value="${gazebo}"/>
     </xacro:include>
   </xacro:if>
   <!-- Left End Effector -->
-  <xacro:include filename="$(find baxter_description)/urdf/left_end_effector.urdf.xacro">
-      <xacro:arg name="left_electric_gripper" value="${left_electric_gripper}"/>
-  </xacro:include>
+  <xacro:include filename="$(find baxter_description)/urdf/left_end_effector.urdf.xacro" />
   <!-- Right End Effector -->
-  <xacro:include filename="$(find baxter_description)/urdf/right_end_effector.urdf.xacro">
-      <xacro:arg name="right_electric_gripper" value="${right_electric_gripper}"/>
-  </xacro:include>
+  <xacro:include filename="$(find baxter_description)/urdf/right_end_effector.urdf.xacro" />
 </robot>

File: src/baxter/baxter_common/baxter_description/urdf/baxter_base/baxter_base.gazebo.xacro (robot description, xacro)
@@ -5,12 +5,9 @@
     <plugin name="baxter_ros_control" filename="libbaxter_gazebo_ros_control.so">
       <robotNamespace>/robot</robotNamespace>
-      <robotSimType>gazebo_ros_control/DefaultRobotHWSim</robotSimType> <!-- Gazebo Default -->
-      <legacyModeNS>true</legacyModeNS>
-      <controlPeriod>0.001</controlPeriod> <!-- Gazebo Default -->
     </plugin>
   </gazebo>
   <!-- Gazebo-Specific Link Properties -->
   <gazebo reference="torso">
-    <self_collide>true</self_collide>
+    <selfCollide>true</selfCollide>
   </gazebo>
   <gazebo reference="head_pan">
@@ -94,8 +91,4 @@
         <distortionT1>0.0</distortionT1>
         <distortionT2>0.0</distortionT2>
-        <CxPrime>0</CxPrime>
-        <Cx>0.0</Cx>
-        <Cy>0.0</Cy>
-        <focalLength>0.0</focalLength>
         <robotNamespace>/cameras</robotNamespace>
       </plugin>
@@ -136,8 +129,4 @@
         <distortionT1>0.0</distortionT1>
         <distortionT2>0.0</distortionT2>
-        <CxPrime>0</CxPrime>
-        <Cx>0.0</Cx>
-        <Cy>0.0</Cy>
-        <focalLength>0.0</focalLength>
         <robotNamespace>/cameras</robotNamespace>
       </plugin>
@@ -178,8 +167,4 @@
         <distortionT1>0.0</distortionT1>
         <distortionT2>0.0</distortionT2>
-        <CxPrime>0</CxPrime>
-        <Cx>0.0</Cx>
-        <Cy>0.0</Cy>
-        <focalLength>0.0</focalLength>
         <robotNamespace>/cameras</robotNamespace>
       </plugin>
@@ -192,5 +177,4 @@
         <width>1024</width>
         <topicName>/robot/xdisplay</topicName>
-        <robotNamespace>/robot</robotNamespace>
       </plugin>
     </visual>
@@ -225,5 +209,4 @@
         <topicName>/robot/sonar/head_sonar/state</topicName>
         <frameName>sonar_ring</frameName>
-        <hokuyoMinIntensity>101</hokuyoMinIntensity>
       </plugin>
       <always_on>true</always_on>
@@ -292,8 +275,8 @@
     <type>transmission_interface/SimpleTransmission</type>
     <joint name="right_s0">
-      <hardwareInterface>hardware_interface/EffortJointInterface</hardwareInterface>
+      <hardwareInterface>EffortJointInterface</hardwareInterface>
     </joint>
     <actuator name="right_motor1">
-      <hardwareInterface>hardware_interface/EffortJointInterface</hardwareInterface>
+      <hardwareInterface>EffortJointInterface</hardwareInterface>
       <mechanicalReduction>1</mechanicalReduction>
     </actuator>
@@ -302,8 +285,8 @@
     <type>transmission_interface/SimpleTransmission</type>
     <joint name="right_s1">
-      <hardwareInterface>hardware_interface/EffortJointInterface</hardwareInterface>
+      <hardwareInterface>EffortJointInterface</hardwareInterface>
     </joint>
     <actuator name="right_motor2">
-      <hardwareInterface>hardware_interface/EffortJointInterface</hardwareInterface>
+      <hardwareInterface>EffortJointInterface</hardwareInterface>
       <mechanicalReduction>1</mechanicalReduction>
     </actuator>
@@ -312,8 +295,8 @@
     <type>transmission_interface/SimpleTransmission</type>
     <joint name="right_e0">
-      <hardwareInterface>hardware_interface/EffortJointInterface</hardwareInterface>
+      <hardwareInterface>EffortJointInterface</hardwareInterface>
     </joint>
     <actuator name="right_motor3">
-      <hardwareInterface>hardware_interface/EffortJointInterface</hardwareInterface>
+      <hardwareInterface>EffortJointInterface</hardwareInterface>
       <mechanicalReduction>1</mechanicalReduction>
     </actuator>
@@ -322,8 +305,8 @@
     <type>transmission_interface/SimpleTransmission</type>
     <joint name="right_e1">
-      <hardwareInterface>hardware_interface/EffortJointInterface</hardwareInterface>
+      <hardwareInterface>EffortJointInterface</hardwareInterface>
     </joint>
     <actuator name="right_motor4">
-      <hardwareInterface>hardware_interface/EffortJointInterface</hardwareInterface>
+      <hardwareInterface>EffortJointInterface</hardwareInterface>
       <mechanicalReduction>1</mechanicalReduction>
     </actuator>
@@ -332,8 +315,8 @@
     <type>transmission_interface/SimpleTransmission</type>
     <joint name="right_w0">
-      <hardwareInterface>hardware_interface/EffortJointInterface</hardwareInterface>
+      <hardwareInterface>EffortJointInterface</hardwareInterface>
     </joint>
     <actuator name="right_motor5">
-      <hardwareInterface>hardware_interface/EffortJointInterface</hardwareInterface>
+      <hardwareInterface>EffortJointInterface</hardwareInterface>
       <mechanicalReduction>1</mechanicalReduction>
     </actuator>
@@ -342,8 +325,8 @@
     <type>transmission_interface/SimpleTransmission</type>
     <joint name="right_w1">
-      <hardwareInterface>hardware_interface/EffortJointInterface</hardwareInterface>
+      <hardwareInterface>EffortJointInterface</hardwareInterface>
     </joint>
     <actuator name="right_motor6">
-      <hardwareInterface>hardware_interface/EffortJointInterface</hardwareInterface>
+      <hardwareInterface>EffortJointInterface</hardwareInterface>
       <mechanicalReduction>1</mechanicalReduction>
     </actuator>
@@ -352,8 +335,8 @@
     <type>transmission_interface/SimpleTransmission</type>
     <joint name="right_w2">
-      <hardwareInterface>hardware_interface/EffortJointInterface</hardwareInterface>
+      <hardwareInterface>EffortJointInterface</hardwareInterface>
     </joint>
     <actuator name="right_motor7">
-      <hardwareInterface>hardware_interface/EffortJointInterface</hardwareInterface>
+      <hardwareInterface>EffortJointInterface</hardwareInterface>
       <mechanicalReduction>1</mechanicalReduction>
     </actuator>
@@ -363,8 +346,8 @@
     <type>transmission_interface/SimpleTransmission</type>
     <joint name="left_s0">
-      <hardwareInterface>hardware_interface/EffortJointInterface</hardwareInterface>
+      <hardwareInterface>EffortJointInterface</hardwareInterface>
     </joint>
     <actuator name="left_motor1">
-      <hardwareInterface>hardware_interface/EffortJointInterface</hardwareInterface>
+      <hardwareInterface>EffortJointInterface</hardwareInterface>
       <mechanicalReduction>1</mechanicalReduction>
     </actuator>
@@ -373,8 +356,8 @@
     <type>transmission_interface/SimpleTransmission</type>
     <joint name="left_s1">
-      <hardwareInterface>hardware_interface/EffortJointInterface</hardwareInterface>
+      <hardwareInterface>EffortJointInterface</hardwareInterface>
     </joint>
     <actuator name="left_motor2">
-      <hardwareInterface>hardware_interface/EffortJointInterface</hardwareInterface>
+      <hardwareInterface>EffortJointInterface</hardwareInterface>
       <mechanicalReduction>1</mechanicalReduction>
     </actuator>
@@ -383,8 +366,8 @@
     <type>transmission_interface/SimpleTransmission</type>
     <joint name="left_e0">
-      <hardwareInterface>hardware_interface/EffortJointInterface</hardwareInterface>
+      <hardwareInterface>EffortJointInterface</hardwareInterface>
     </joint>
     <actuator name="left_motor3">
-      <hardwareInterface>hardware_interface/EffortJointInterface</hardwareInterface>
+      <hardwareInterface>EffortJointInterface</hardwareInterface>
       <mechanicalReduction>1</mechanicalReduction>
     </actuator>
@@ -393,8 +376,8 @@
     <type>transmission_interface/SimpleTransmission</type>
     <joint name="left_e1">
-      <hardwareInterface>hardware_interface/EffortJointInterface</hardwareInterface>
+      <hardwareInterface>EffortJointInterface</hardwareInterface>
     </joint>
     <actuator name="left_motor4">
-      <hardwareInterface>hardware_interface/EffortJointInterface</hardwareInterface>
+      <hardwareInterface>EffortJointInterface</hardwareInterface>
       <mechanicalReduction>1</mechanicalReduction>
     </actuator>
@@ -403,8 +386,8 @@
     <type>transmission_interface/SimpleTransmission</type>
     <joint name="left_w0">
-      <hardwareInterface>hardware_interface/EffortJointInterface</hardwareInterface>
+      <hardwareInterface>EffortJointInterface</hardwareInterface>
     </joint>
     <actuator name="left_motor5">
-      <hardwareInterface>hardware_interface/EffortJointInterface</hardwareInterface>
+      <hardwareInterface>EffortJointInterface</hardwareInterface>
       <mechanicalReduction>1</mechanicalReduction>
     </actuator>
@@ -413,8 +396,8 @@
     <type>transmission_interface/SimpleTransmission</type>
     <joint name="left_w1">
-      <hardwareInterface>hardware_interface/EffortJointInterface</hardwareInterface>
+      <hardwareInterface>EffortJointInterface</hardwareInterface>
     </joint>
     <actuator name="left_motor6">
-      <hardwareInterface>hardware_interface/EffortJointInterface</hardwareInterface>
+      <hardwareInterface>EffortJointInterface</hardwareInterface>
       <mechanicalReduction>1</mechanicalReduction>
     </actuator>
@@ -423,8 +406,8 @@
     <type>transmission_interface/SimpleTransmission</type>
     <joint name="left_w2">
-      <hardwareInterface>hardware_interface/EffortJointInterface</hardwareInterface>
+      <hardwareInterface>EffortJointInterface</hardwareInterface>
     </joint>
     <actuator name="left_motor7">
-      <hardwareInterface>hardware_interface/EffortJointInterface</hardwareInterface>
+      <hardwareInterface>EffortJointInterface</hardwareInterface>
       <mechanicalReduction>1</mechanicalReduction>
     </actuator>
@@ -434,8 +417,8 @@
     <type>transmission_interface/SimpleTransmission</type>
     <joint name="head_pan">
-      <hardwareInterface>hardware_interface/EffortJointInterface</hardwareInterface>
+      <hardwareInterface>EffortJointInterface</hardwareInterface>
     </joint>
     <actuator name="head_motor1">
-      <hardwareInterface>hardware_interface/EffortJointInterface</hardwareInterface>
+      <hardwareInterface>EffortJointInterface</hardwareInterface>
       <mechanicalReduction>1</mechanicalReduction>
     </actuator>

File: src/baxter/baxter_common/baxter_description/urdf/left_end_effector.urdf.xacro (robot description, xacro)
@@ -1,20 +1,13 @@
 <?xml version="1.0" ?>
-<robot name="left_end_effector" xmlns:xacro="http://ros.org/wiki/xacro">
-  <xacro:arg name="left_electric_gripper" default="false"/>
-  <xacro:if value="$(arg left_electric_gripper)">
-    <xacro:include filename="$(find rethink_ee_description)/urdf/electric_gripper/rethink_electric_gripper.xacro" />
-    <xacro:rethink_electric_gripper side="left"
-                                    l_finger="standard_narrow"
-                                    l_finger_slot="1"
-                                    l_finger_tip="basic_soft_tip"
-                                    l_finger_grasp="inner"
-                                    r_finger="standard_narrow"
-                                    r_finger_slot="1"
-                                    r_finger_tip="basic_soft_tip"
-                                    r_finger_grasp="inner"/>
-  </xacro:if>
-  <xacro:unless value="$(arg left_electric_gripper)">
-  <xacro:include filename="$(cwd)/src/baxter/baxter_common/rethink_ee_description/urdf/null_gripper/null_gripper.xacro" />
-    <xacro:null_gripper side="left"/>
-  </xacro:unless>
+<robot name="left_end_effector" xmlns:xacro="http://www.ros.org/wiki/xacro">
+  <xacro:include filename="$(find rethink_ee_description)/urdf/electric_gripper/rethink_electric_gripper.xacro" />
+  <xacro:rethink_electric_gripper side="left"
+                                  l_finger="extended_narrow"
+                                  l_finger_slot="2"
+                                  l_finger_tip="paddle_tip"
+                                  l_finger_grasp="inner"
+                                  r_finger="extended_narrow"
+                                  r_finger_slot="2"
+                                  r_finger_tip="paddle_tip"
+                                  r_finger_grasp="inner"/>
 </robot>

File: src/baxter/baxter_common/baxter_description/urdf/right_end_effector.urdf.xacro (robot description, xacro)
@@ -1,20 +1,13 @@
 <?xml version="1.0" ?>
-<robot name="right_end_effector" xmlns:xacro="http://ros.org/wiki/xacro">
-  <xacro:arg name="right_electric_gripper" default="false"/>
-  <xacro:if value="$(arg right_electric_gripper)">
-    <xacro:include filename="$(find rethink_ee_description)/urdf/electric_gripper/rethink_electric_gripper.xacro" />
-    <xacro:rethink_electric_gripper side="right"
-                                    l_finger="extended_wide"
-                                    l_finger_slot="4"
-                                    l_finger_tip="paddle_tip"
-                                    l_finger_grasp="inner"
-                                    r_finger="extended_wide"
-                                    r_finger_slot="4"
-                                    r_finger_tip="paddle_tip"
-                                    r_finger_grasp="inner"/>
-  </xacro:if>
-  <xacro:unless value="$(arg right_electric_gripper)">
-  <xacro:include filename="$(cwd)/src/baxter/baxter_common/rethink_ee_description/urdf/null_gripper/null_gripper.xacro" />
-    <xacro:null_gripper side="right"/>
-  </xacro:unless>
+<robot name="right_end_effector" xmlns:xacro="http://www.ros.org/wiki/xacro">
+  <xacro:include filename="$(find rethink_ee_description)/urdf/electric_gripper/rethink_electric_gripper.xacro" />
+  <xacro:rethink_electric_gripper side="right"
+                                  l_finger="extended_narrow"
+                                  l_finger_slot="2"
+                                  l_finger_tip="half_round_tip"
+                                  l_finger_grasp="inner"
+                                  r_finger="extended_narrow"
+                                  r_finger_slot="2"
+                                  r_finger_tip="half_round_tip"
+                                  r_finger_grasp="inner"/>
 </robot>
